Commit message: chore: 修改了attachlink的偏移量和抓取位置的计算参数

File: src/my_robot_description/urdf/gripper.xacro (robot description, xacro)
@@ -99,5 +99,5 @@
         <parent link="gripper_base_link" />
         <child link="attach_link" />
-        <origin xyz="0 0 0.02" rpy="0 0 0" />
+        <origin xyz="0 0 0.022" rpy="0 0 0" />
     </joint>
     <gazebo reference="gripper_attach_joint">
